File: proyectofinal/proyectofinal.kicad_sch (KiCad schematic)
At the start: 7 parts, among them J2 conector paramodulo lora, J3 dht22, J4 Guva-s12s, J5 convertidor_TTL, U1 ESP32_NODEMCU, U3 mp1584

Commit message: minimas
minimas
Parts:
- removed U1: ESP32_NODEMCU, ESP32_NODEMCU:MODULE_ESP32_NODEMCU, symbol ESP32_NODEMCU:ESP32_NODEMCU
- removed U3: mp1584, MP1584EN-master:SRT_MPT1584EN_Module, symbol New_Library:mp1584
- added C1, C3: 100uf/25v, Capacitor_THT:CP_Radial_D6.3mm_P2.50mm, symbol Device:C_Polarized
- added C2, C4: 10uf/25v, Capacitor_THT:CP_Radial_D5.0mm_P2.50mm, symbol Device:C_Polarized
- added J1: cnn, Connector_AMASS:AMASS_XT60-F_1x02_P7.20mm_Vertical, symbol Connector:Conn_01x02_Socket
- added U1: LM7833_TO220, Package_TO_SOT_THT:TO-220-3_Vertical, symbol Regulator_Linear:LM7805_TO220
- added U2: ESP32_DevKit_V1_DOIT, esp32_devkit_v1_doit:esp32_devkit_v1_doit, symbol esp32_devkit_v1_doit:ESP32_DevKit_V1_DOIT
- added U3: LM7805_TO220, Package_TO_SOT_THT:TO-220-3_Vertical, symbol Regulator_Linear:LM7805_TO220
Connections:
- net +3.3V: now also J3.2 (Pin_2), R1.2, C2.1, U1.3 (VO); no longer J3.1 (Pin_1), J5.5 (Pin_5), R1.1
- net +5V: now also J5.5 (Pin_5), C1.1, C4.1, U1.1 (VI), U2.15 (VIN), U3.3 (VO)
- net DE/RE_TTL: now also U2.26 (IO21)
- net DI_TTL: now also U2.28 (TXD0/IO1)
- net GND: now also C1.2, C2.2, C3.2, C4.2, J1.2 (Pin_2), U1.2 (GND), U2.14 (GND), U2.17 (GND), U3.2 (GND)
- net IRQ_SPI_LoRa: now also U2.22 (IO17)
- net MISO_SPI_LoRa: now also U2.25 (IO19)
- net MOSI_SPI_LoRa: now also U2.30 (IO23)
- net NSS_SPI_LoRa: now also U2.23 (IO5)
- net RO_TTL: now also U2.27 (RXD0/IO3)
- net RST_LoRa: now also U2.21 (IO16)
- net SCK_CLOCK_SPI_LoRa: now also U2.24 (IO18)
- net SIG_DHT22: now also J3.1 (Pin_1), R1.1; no longer J3.2 (Pin_2), R1.2
- new net: C3.1, J1.1 (Pin_1), U3.1 (VI)

Commit message: e
e
Connections:
- net GND: now also J3.3 (Pin_3); no longer J3.4 (Pin_4)
- net SIG_DHT22: now also J3.4 (Pin_4), U2.7 (IO33); no longer J3.1 (Pin_1)
- net SIG_Guva-s12s: now also U2.6 (IO32)
Other:
- moved on the sheet: J3, R1
Changed lines of the file:
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@@
-	)
-	(junction
-		(at 66.04 95.25)
-		(diameter 0)
-		(color 0 0 0 0)
 	)
 	(junction
@@
 	)
 	(junction
+		(at 62.23 97.79)
+		(diameter 0)
+		(color 0 0 0 0)
+	)
+	(junction
 		(at 55.88 55.88)
 		(diameter 0)
@@
 	)
 	(junction
-		(at 66.04 87.63)
+		(at 62.23 105.41)
 		(diameter 0)
 		(color 0 0 0 0)
@@
 	)
 	(no_connect
-		(at 57.15 97.79)
+		(at 53.34 92.71)
 	)
 	(no_connect
@@
 	(wire
 		(pts
-			(xy 69.85 86.36) (xy 69.85 87.63)
+			(xy 66.04 106.68) (xy 66.04 105.41)
 		)
 		(stroke
@@
 	(wire
 		(pts
-			(xy 71.12 86.36) (xy 69.85 86.36)
-		)
-		(stroke
-			(width 0)
-			(type default)
-		)
-	)
-	(wire
-		(pts
-			(xy 63.5 92.71) (xy 63.5 87.63)
+			(xy 67.31 106.68) (xy 66.04 106.68)
+		)
+		(stroke
+			(width 0)
+			(type default)
+		)
+	)
+	(wire
+		(pts
+			(xy 59.69 100.33) (xy 59.69 105.41)
 		)
 		(stroke
@@
 	(wire
 		(pts
-			(xy 57.15 95.25) (xy 66.04 95.25)
-		)
-		(stroke
-			(width 0)
-			(type default)
-		)
-	)
-	(wire
-		(pts
 			(xy 60.96 49.53) (xy 55.88 49.53)
 		)
@@
 	(wire
 		(pts
+			(xy 58.42 96.52) (xy 53.34 96.52)
+		)
+		(stroke
+			(width 0)
+			(type default)
+		)
+	)
+	(wire
+		(pts
 			(xy 55.88 54.61) (xy 55.88 55.88)
 		)
@@
 	(wire
 		(pts
-			(xy 66.04 95.25) (xy 77.47 95.25)
-		)
-		(stroke
-			(width 0)
-			(type default)
-		)
-	)
-	(wire
-		(pts
-			(xy 58.42 100.33) (xy 57.15 100.33)
+			(xy 62.23 97.79) (xy 73.66 97.79)
 		)
 		(stroke
@@
 	(wire
 		(pts
-			(xy 63.5 87.63) (xy 66.04 87.63)
+			(xy 59.69 105.41) (xy 62.23 105.41)
 		)
 		(stroke
@@
 	(wire
 		(pts
-			(xy 57.15 92.71) (xy 63.5 92.71)
+			(xy 53.34 96.52) (xy 53.34 97.79)
+		)
+		(stroke
+			(width 0)
+			(type default)
+		)
+	)
+	(wire
+		(pts
+			(xy 53.34 100.33) (xy 59.69 100.33)
+		)
+		(stroke
+			(width 0)
+			(type default)
+		)
+	)
+	(wire
+		(pts
+			(xy 53.34 95.25) (xy 62.23 95.25)
 		)
 		(stroke
@@
 	(wire
 		(pts
+			(xy 62.23 95.25) (xy 62.23 97.79)
+		)
+		(stroke
+			(width 0)
+			(type default)
+		)
+	)
+	(wire
+		(pts
 			(xy 186.69 72.39) (xy 191.77 72.39)
 		)
@@
 	(wire
 		(pts
-			(xy 69.85 87.63) (xy 66.04 87.63)
+			(xy 66.04 105.41) (xy 62.23 105.41)
 		)
 		(stroke
@@
 	(global_label "SIG_DHT22"
 		(shape input)
-		(at 71.12 86.36 0)
+		(at 67.31 106.68 0)
 		(fields_autoplaced yes)
 		(effects
@@
 		)
 		(property "Intersheetrefs" "${INTERSHEET_REFS}"
-			(at 84.1442 86.36 0)
+			(at 80.3342 106.68 0)
 			(effects
 				(font
@@
 	(global_label "SIG_Guva-s12s"
 		(shape input)
-		(at 151.13 109.22 0)
+		(at 134.62 106.68 0)
 		(fields_autoplaced yes)
 		(effects
@@
 		)
 		(property "Intersheetrefs" "${INTERSHEET_REFS}"
-			(at 168.327 109.22 0)
+			(at 151.817 106.68 0)
 			(effects
 				(font
@@
 		)
 	)
-	(global_label "SIG_DHT22"
+	(global_label "SCK_CLOCK_SPI_LoRa"
 		(shape input)
-		(at 151.13 111.76 0)
+		(at 55.88 125.73 0)
 		(fields_autoplaced yes)
 		(effects
@@
 		)
 		(property "Intersheetrefs" "${INTERSHEET_REFS}"
-			(at 164.1542 111.76 0)
-			(effects
-				(font
-					(size 1.27 1.27)
-				)
-				(justify left)
-				(hide yes)
-			)
-		)
-	)
-	(global_label "SCK_CLOCK_SPI_LoRa"
+			(at 79.3665 125.73 0)
+			(effects
+				(font
+					(size 1.27 1.27)
+				)
+				(justify left)
+				(hide yes)
+			)
+		)
+	)
+	(global_label "MISO_SPI_LoRa"
 		(shape input)
-		(at 55.88 125.73 0)
+		(at 55.88 130.81 0)
 		(fields_autoplaced yes)
 		(effects
@@
 		)
 		(property "Intersheetrefs" "${INTERSHEET_REFS}"
-			(at 79.3665 125.73 0)
-			(effects
-				(font
-					(size 1.27 1.27)
-				)
-				(justify left)
-				(hide yes)
-			)
-		)
-	)
-	(global_label "MISO_SPI_LoRa"
+			(at 73.077 130.81 0)
+			(effects
+				(font
+					(size 1.27 1.27)
+				)
+				(justify left)
+				(hide yes)
+			)
+		)
+	)
+	(global_label "SIG_DHT22"
 		(shape input)
-		(at 55.88 130.81 0)
+		(at 134.62 109.22 0)
 		(fields_autoplaced yes)
 		(effects
@@
 		)
 		(property "Intersheetrefs" "${INTERSHEET_REFS}"
-			(at 73.077 130.81 0)
+			(at 147.6442 109.22 0)
 			(effects
 				(font
@@
 	(symbol
 		(lib_id "Connector:Conn_01x04_Pin")
-		(at 52.07 95.25 0)
+		(at 48.26 95.25 0)
 		(unit 1)
 		(exclude_from_sim no)
@@
 		(fields_autoplaced yes)
 		(property "Reference" "J3"
-			(at 52.705 87.63 0)
+			(at 48.895 87.63 0)
 			(effects
 				(font
@@
 		)
 		(property "Value" "dht22"
-			(at 52.705 90.17 0)
+			(at 48.895 90.17 0)
 			(effects
 				(font
@@
 		)
 		(property "Footprint" "Connector_Molex:Molex_KK-254_AE-6410-04A_1x04_P2.54mm_Vertical"
-			(at 52.07 95.25 0)
+			(at 48.26 95.25 0)
 			(effects
 				(font
@@
 		)
 		(property "Datasheet" "~"
-			(at 52.07 95.25 0)
+			(at 48.26 95.25 0)
 			(effects
 				(font
@@
 		)
 		(property "Description" "Generic connector, single row, 01x04, script generated"
-			(at 52.07 95.25 0)
+			(at 48.26 95.25 0)
 			(effects
 				(font
@@
 		)
 		(instances
-			(project ""
+			(project "proyectofinal"
 				(path "/e7d7c171-9d86-45d9-a9f9-7abd3dbd6a53"
 					(reference "J3")
@@
 	(symbol
 		(lib_id "power:GND")
-		(at 58.42 100.33 0)
+		(at 58.42 96.52 0)
 		(unit 1)
 		(exclude_from_sim no)
@@
 		(fields_autoplaced yes)
 		(property "Reference" "#PWR06"
-			(at 58.42 106.68 0)
+			(at 58.42 102.87 0)
 			(effects
 				(font
@@
 		)
 		(property "Value" "GND"
-			(at 58.42 105.41 0)
+			(at 58.42 101.6 0)
 			(effects
 				(font
@@
 		)
 		(property "Footprint" ""
-			(at 58.42 100.33 0)
+			(at 58.42 96.52 0)
 			(effects
 				(font
@@
 		)
 		(property "Datasheet" ""
-			(at 58.42 100.33 0)
+			(at 58.42 96.52 0)
 			(effects
 				(font
@@
 		)
 		(property "Description" "Power symbol creates a global label with name \"GND\" , ground"
-			(at 58.42 100.33 0)
+			(at 58.42 96.52 0)
 			(effects
 				(font
@@
 	(symbol
 		(lib_id "Device:R")
-		(at 66.04 91.44 0)
+		(at 62.23 101.6 0)
+		(mirror x)
 		(unit 1)
 		(exclude_from_sim no)
@@
 		(fields_autoplaced yes)
 		(property "Reference" "R1"
-			(at 68.58 90.1699 0)
+			(at 64.77 102.8701 0)
 			(effects
 				(font
@@
 		)
 		(property "Value" "30k"
-			(at 68.58 92.7099 0)
+			(at 64.77 100.3301 0)
 			(effects
 				(font
@@
 		)
 		(property "Footprint" "Resistor_THT:R_Axial_DIN0207_L6.3mm_D2.5mm_P10.16mm_Horizontal"
-			(at 64.262 91.44 90)
+			(at 60.452 101.6 90)
 			(effects
 				(font
@@
 		)
 		(property "Datasheet" "~"
-			(at 66.04 91.44 0)
+			(at 62.23 101.6 0)
 			(effects
 				(font
@@
 		)
 		(property "Description" "Resistor"
-			(at 66.04 91.44 0)
+			(at 62.23 101.6 0)
 			(effects
 				(font
@@
 	(symbol
 		(lib_id "power:+3.3V")
-		(at 77.47 95.25 0)
+		(at 73.66 97.79 0)
+		(mirror x)
 		(unit 1)
 		(exclude_from_sim no)
@@
 		(fields_autoplaced yes)
 		(property "Reference" "#PWR05"
-			(at 77.47 99.06 0)
+			(at 73.66 93.98 0)
 			(effects
 				(font
@@
 		)
 		(property "Value" "+3.3V"
-			(at 77.47 90.17 0)
+			(at 73.66 102.87 0)
 			(effects
 				(font
@@
 		)
 		(property "Footprint" ""
-			(at 77.47 95.25 0)
+			(at 73.66 97.79 0)
 			(effects
 				(font
@@
 		)
 		(property "Datasheet" ""
-			(at 77.47 95.25 0)
+			(at 73.66 97.79 0)
 			(effects
 				(font
@@
 		)
 		(property "Description" "Power symbol creates a global label with name \"+3.3V\""
-			(at 77.47 95.25 0)
-			(effects
-				(font
+			(at 73.66 97.79 0)
+			(effects
+				(font

Commit message: e
e
Parts:
- removed J2: conector paramodulo lora, Connector_Molex:Molex_SL_171971-0012_1x12_P2.54mm_Vertical, symbol Connector:Conn_01x12_Pin
- removed U2: ESP32_DevKit_V1_DOIT, esp32_devkit_v1_doit:esp32_devkit_v1_doit, symbol esp32_devkit_v1_doit:ESP32_DevKit_V1_DOIT
- added J2: conector alimentacion esp, Connector_JST:JST_EH_B2B-EH-A_1x02_P2.50mm_Vertical, symbol Connector:Conn_01x02_Socket
- added J6: MICS-6814, Connector_Molex:Molex_KK-254_AE-6410-05A_1x05_P2.54mm_Vertical, symbol Connector:Conn_01x05_Pin
- added K1, K2: SRD-05VDC-SL-C, SRD-05VDC-SL-C:RELAY_SRD-05VDC-SL-C, symbol SRD-05VDC-SL-C:SRD-05VDC-SL-C
- added U4: ESP32_LORA_V2.0, ESP32_LORA_V2.0:MODULE_ESP32_LORA_V2.0, symbol ESP32_LORA_V2.0:ESP32_LORA_V2.0
Connections:
- net +3.3V: now also J2.1 (Pin_1), K1.NO; no longer J3.2 (Pin_2), J4.1 (Pin_1), R1.2
- net +5V: now also K2.NO; no longer J5.5 (Pin_5)
- net DE/RE_TTL: now also U4.J2_9 (UO_RTS/V_SPI_QP/GPIO22/SCL/22)
- net DI_TTL: now also U4.J2_17 (U2_TXD/GPIO17/17)
- net GND: now also J2.2 (Pin_2), J6.5 (Pin_5), K1.A2, K1.NC, K2.A2, K2.NC
- net RO_TTL: now also U4.J2_18 (OLED_RST/U2_RXD/GPIO16/16)
- net SIG_DHT22: now also U4.J3_16 (TOUCH5/ADC2_5/GPIO12/12)
- net SIG_Guva-s12s: now also U4.J3_12 (LED/DAC2/ADC2_8/GPIO25/25)
- new net: U4. (GND), U4.J3_1 (GND)
- new net: U4. (GND), U4.J3_3 (3V3)
- new net +3.3V sensores: J3.2 (Pin_2), J4.1 (Pin_1), K1.COM, R1.2
- new net +5V sensores: J5.5 (Pin_5), J6.4 (Pin_4), K2.COM
- new net SIG_Co_MICS-6814: J6.1 (Pin_1), U4.J2_8 (PRG_BUTTON/TOUCH1/ADC2_1/GPIO0/0)
- new net SIG_N02_MICS-6814: J6.3 (Pin_3), U4.J3_17 (TOUCH4/ADC2_4/GPIO13/13)
- new net SIG_NH3_MICS-6814: J6.2 (Pin_2), U4.J2_15 (TOUCH2/HSPI_WP/ADC2_2/GPIO2/2)
- new net vext: K1.A1, K2.A1, U4. (GND), U4.J2_4 (VEXT)
- no-connect marks 4 -> 1
Other:
- note added: "alimentacion"
- note added: "sensores"
- moved on the sheet: C1, C2, C3, C4, J1, J3, J4, J5, R1, U1, U3

Commit message: w
w
Other:
- note added: "microcontrolador"
- moved on the sheet: C1, C2, C3, C4, J1, J2, J3, J4, J5, J6, K1, K2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
