File: proyectofinal/proyectofinal.kicad_pcb (KiCad board)
At the start: 2 copper layers, 7 parts, among them J2 conector paramodulo lora, J3 dht22, J4 Guva-s12s, J5 convertidor_TTL, U1 ESP32_NODEMCU, U3 mp1584

Commit message: minimas
minimas
Parts:
- added C1: 100uf/25v, Capacitor_THT:CP_Radial_D6.3mm_P2.50mm, F.Cu at (107.0, 83.5)
- added C2: 10uf/25v, Capacitor_THT:CP_Radial_D5.0mm_P2.50mm, F.Cu at (117.0, 76.5)
- added C3: 100uf/25v, Capacitor_THT:CP_Radial_D6.3mm_P2.50mm, F.Cu at (105.5, 98.8)
- added C4: 10uf/25v, Capacitor_THT:CP_Radial_D5.0mm_P2.50mm, F.Cu at (107.0, 90.5)
- added J1: cnn, Connector_AMASS:AMASS_XT60-F_1x02_P7.20mm_Vertical, F.Cu at (97.5, 97.0)
- added U2: ESP32_DevKit_V1_DOIT, esp32_devkit_v1_doit:esp32_devkit_v1_doit, F.Cu at (73.3, 63.1)
- U1: value ESP32_NODEMCU -> LM7833_TO220; footprint ESP32_NODEMCU (1):MODULE_ESP32_NODEMCU -> Package_TO_SOT_THT:TO-220-3_Vertical
- U3: value mp1584 -> LM7805_TO220; footprint MP1584EN-master:SRT_MPT1584EN_Module -> Package_TO_SOT_THT:TO-220-3_Vertical
- moved U3 82.2 mm to (110.5, 98.5)
- moved U1 55.0 mm to (107.0, 77.9)
- moved J2 25.1 mm to (98.5, 88.3)
- moved R1 19.3 mm to (106.4, 71.0), turned to 0 degrees
- moved J4 18.3 mm to (113.5, 64.1)
- moved J3 18.2 mm to (106.5, 66.8)
- moved J5 11.0 mm to (91.5, 71.7)
Connections:
- J3 pad 1: +3.3V -> SIG_DHT22
- J3 pad 2: SIG_DHT22 -> +3.3V
- J5 pad 5: +3.3V -> +5V
- R1 pad 1: +3.3V -> SIG_DHT22
- R1 pad 2: SIG_DHT22 -> +3.3V
- U3 pad 1: VCC -> Net-(J1-Pin_1)
Routing:
- net GND: track 51.2 -> 287.7 mm
- net +5V: track 26.6 -> 181.4 mm
- net +3.3V: track 176.7 -> 38.5 mm
- net DI_TTL: track 135.6 -> 5.92 mm
- net RO_TTL: track 119.9 -> 5.92 mm
- net DE/RE_TTL: track 118.4 -> 20.1 mm
- net MOSI_SPI_LoRa: track 0.00 -> 45.7 mm, vias 0 -> 2
- net Net-(J1-Pin_1): track 0.00 -> 15.2 mm
- net SIG_DHT22: track 9.81 -> 4.23 mm
- net MISO_SPI_LoRa: track 9.56 -> 13.9 mm
- net RST_LoRa: track 8.50 -> 12.6 mm
- net NSS_SPI_LoRa: track 8.50 -> 12.6 mm
- net IRQ_SPI_LoRa: track 8.50 -> 12.6 mm
- net SCK_CLOCK_SPI_LoRa: track 8.50 -> 12.6 mm
- net VCC: track 2.54 -> 0.00 mm

Commit message: e
e
Parts:
- moved R1 19.3 mm to (118.5, 55.9), turned to -90 degrees
Connections:
- J3 pad 1: SIG_DHT22 -> unconnected-(J3-Pin_1-Pad1)
- J3 pad 3: unconnected-(J3-Pin_3-Pad3) -> GND
- J3 pad 4: GND -> SIG_DHT22
- U2 pad 6: unconnected-(U2-IO32-Pad6) -> SIG_Guva-s12s
- U2 pad 7: unconnected-(U2-IO33-Pad7) -> SIG_DHT22
Routing:
- net SIG_Guva-s12s: track 0.00 -> 89.0 mm
- net SIG_DHT22: track 4.23 -> 82.9 mm
- net GND: track 287.7 -> 291.3 mm
- net +3.3V: track 38.5 -> 40.4 mm
- net MOSI_SPI_LoRa: track 45.7 -> 47.0 mm

Commit message: e
e
Parts:
- removed U2: ESP32_DevKit_V1_DOIT, esp32_devkit_v1_doit:esp32_devkit_v1_doit
- added J6: MICS-6814, Connector_Molex:Molex_KK-254_AE-6410-05A_1x05_P2.54mm_Vertical, F.Cu at (216.0, 101.7)
- added K1: SRD-05VDC-SL-C, SRD-05VDC-SL-C:RELAY_SRD-05VDC-SL-C, F.Cu at (202.2, 79.6)
- added K2: SRD-05VDC-SL-C, SRD-05VDC-SL-C:RELAY_SRD-05VDC-SL-C, F.Cu at (218.4, 79.6)
- added U4: ESP32_LORA_V2.0, ESP32_LORA_V2.0:MODULE_ESP32_LORA_V2.0, F.Cu at (178.8, 80.8)
- J2: value conector paramodulo lora -> conector alimentacion esp; footprint Connector_Molex:Molex_SL_171971-0012_1x12_P2.54mm_Vertical -> Connector_JST:JST_EH_B2B-EH-A_1x02_P2.50mm_Vertical
- moved J5 135.5 mm to (223.0, 104.2)
- moved C4 116.0 mm to (219.9, 63.9), turned to -90 degrees
- moved U1 115.5 mm to (220.8, 58.4)
- moved C2 108.9 mm to (225.2, 63.9), turned to -90 degrees
- moved C1 108.6 mm to (213.9, 63.9), turned to -90 degrees
- moved J1 108.5 mm to (198.7, 57.9)
- moved U3 107.7 mm to (210.4, 58.5), turned to 0 degrees
- moved C3 107.5 mm to (207.2, 63.9)
- moved R1 102.7 mm to (210.8, 101.0), turned to 90 degrees
- moved J3 102.1 mm to (205.6, 91.5), turned to -90 degrees
- moved J4 89.4 mm to (198.5, 91.5), turned to -90 degrees
- moved J2 86.7 mm to (177.5, 52.5), turned to 0 degrees
Connections:
- J2 pad 1: GND -> +3.3V
- J2 pad 2: RST_LoRa -> GND
- J3 pad 2: +3.3V -> +3.3V sensores
- J4 pad 1: +3.3V -> +3.3V sensores
- J5 pad 5: +5V -> +5V sensores
- R1 pad 2: +3.3V -> +3.3V sensores
Routing:
- net +5V: track 181.4 -> 46.2 mm
- net GND: track 291.3 -> 176.8 mm
- net DE/RE_TTL: track 20.1 -> 124.5 mm
- net +3.3V: track 40.4 -> 123.6 mm
- net vext: track 0.00 -> 80.1 mm
- net DI_TTL: track 5.92 -> 83.9 mm
- net SIG_Guva-s12s: track 89.0 -> 15.2 mm
- net SIG_Co_MICS-6814: track 0.00 -> 72.7 mm
- net SIG_NH3_MICS-6814: track 0.00 -> 66.0 mm
- net SIG_DHT22: track 82.9 -> 22.3 mm
- net RO_TTL: track 5.92 -> 63.0 mm
- net MOSI_SPI_LoRa: track 47.0 -> 0.00 mm, vias 2 -> 0
- net SIG_N02_MICS-6814: track 0.00 -> 33.0 mm
- net +3.3V sensores: track 0.00 -> 18.7 mm
- net +5V sensores: track 0.00 -> 14.0 mm
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Other:
- board outline added: 72.5 x 67 mm

Commit message: s
s
Parts:
- K1: value SRD-05VDC-SL-C -> rele 3.3v
- K2: value SRD-05VDC-SL-C -> rele 5v
- moved U3 0.37 mm to (210.1, 58.4)
Changed lines of the file:
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@@
 	(footprint "Package_TO_SOT_THT:TO-220-3_Vertical"
 		(layer "F.Cu")
-		(at 210.45 58.465)
+		(at 210.085 58.4)
 		(descr "TO-220-3, Vertical, RM 2.54mm, see https://www.vishay.com/docs/66542/to-220-1.pdf, generated with kicad-footprint-generator TO_SOT_THT_generate.py")
 		(tags "TO-220-3 Vertical RM 2.54mm")
@@
 		)
 		(property "Value" "Guva-s12s"
-			(at 7.92 -0.575 0)
+			(at 7.875 0.47 0)
 			(layer "F.Fab")
 			(effects
@@
 		)
 		(property "Value" "MICS-6814"
-			(at -5.26 0 0)
+			(at -2.84 -1.03 0)
 			(layer "F.Fab")
 			(effects
@@
 		)
 		(property "Value" "10uf/25v"
-			(at -2.794888 0 0)
+			(at 4.890112 0.058211 0)
 			(layer "F.Fab")
 			(effects
@@
 		)
 		(property "Value" "dht22"
-			(at 10.42 0 0)
+			(at 10.45 -0.065 0)
 			(layer "F.Fab")
 			(effects
@@
 		)
 		(property "Value" "convertidor_TTL"
-			(at -6.92 0.1625 0)
+			(at -2.625 0.03 0)
 			(layer "F.Fab")
 			(effects
@@
 			)
 		)
-		(property "Value" "SRD-05VDC-SL-C"
-			(at 14.644888 88.644404 180)
+		(property "Value" "rele 3.3v"
+			(at 0.0275 0.21 180)
 			(layer "F.Fab")
 			(effects
@@
 			)
 		)
-		(property "Value" "SRD-05VDC-SL-C"
-			(at 11.115 3.775 180)
+		(property "Value" "rele 5v"
+			(at -0.2475 0.385 180)
 			(layer "F.Fab")
 			(effects
@@
 	)
 	(segment
+		(start 212.5385 55.599)
+		(end 209.4895 52.55)
+		(width 1)
+		(layer "B.Cu")
+		(net 2)
+	)
+	(segment
 		(start 222.55 60.715)
 		(end 222.55 66.409888)
@@
 	)
 	(segment
-		(start 212.99 56.0505)
-		(end 212.99 58.465)
-		(width 1)
-		(layer "B.Cu")
-		(net 2)
-	)
-	(segment
 		(start 210.375 63.612462)
 		(end 210.375 66.409888)
@@
 	)
 	(segment
-		(start 209.4895 52.55)
-		(end 212.99 56.0505)
-		(width 1)
-		(layer "B.Cu")
-		(net 2)
-	)
-	(segment
 		(start 208.249106 96.605)
 		(end 214.931 89.923106)
@@
 	)
 	(segment
-		(start 212.99 58.465)
-		(end 212.99 60.997462)
+		(start 212.5385 61.448962)
+		(end 212.5385 55.599)
+		(width 1)
+		(layer "B.Cu")
+		(net 2)
+	)
+	(segment
+		(start 210.375 63.612462)
+		(end 212.5385 61.448962)
 		(width 1)
 		(layer "B.Cu")
@@
 		(width 1)
 		(layer "B.Cu")
-		(net 2)
-	)
-	(segment
-		(start 212.99 60.997462)
-		(end 210.375 63.612462)
-		(width 1)
-		(layer "B.Cu")

Commit message: k
l
Parts:
- moved C2 1.79 mm to (227.0, 63.9)
- moved C4 1.14 mm to (221.0, 63.9)
- moved U3 0.67 mm to (209.4, 58.4)
- moved C1 0.63 mm to (214.5, 63.9)
- moved U1 0.20 mm to (221.0, 58.4)
Routing:
- net +3.3V: track 123.6 -> 135.6 mm
- net GND: track 176.4 -> 182.6 mm
- net +5V: track 46.2 -> 51.6 mm
- net vext: track 80.1 -> 81.4 mm
- net Net-(J1-Pin_1): track 16.9 -> 16.1 mm
- net SIG_Guva-s12s: track 15.2 -> 15.8 mm
- net (no net): vias 0 -> 4
- added copper zone on B.Cu, net GND
Other:
- board size 72.5 x 67 mm -> 77 x 67 mm
