File: electronica/proyectofinal/proyectofinal.kicad_pcb (KiCad board)
At the start: 2 copper layers, 77 x 67 mm, 16 parts, among them J1 cnn, J2 conector alimentacion esp, J3 dht22, J4 Guva-s12s, J5 convertidor_TTL, J6 MICS-6814, K1 rele 3.3v, K2 rele 5v, U1 LM7833_TO220, U3 LM7805_TO220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

Commit message: le cambie la resistencia de pullup del dht22
le cambie la resistencia de pullup del dht22
Parts:
- R1: value 30k -> 10k
Changed lines of the file:
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@@
 			(psa4output no)
 			(plot_black_and_white yes)
+			(plotinvisibletext no)
 			(sketchpadsonfab no)
 			(plotpadnumbers no)
@@
 			)
 		)
-		(property "Value" "30k"
+		(property "Value" "10k"
 			(at 5.16 0 90)
 			(layer "F.Fab")
@@
 			(keep_text_aligned yes)
 		)
-		(gr_text "77,025"
+		(gr_text "77.025"
 			(at 198.9375 45.625 0)
 			(layer "Edge.Cuts")

Commit message: loisto
st
Parts:
- removed J6: MICS-6814, Connector_Molex:Molex_KK-254_AE-6410-05A_1x05_P2.54mm_Vertical
- added D1: 1N4007, Diode_THT:D_DO-41_SOD81_P10.16mm_Horizontal, F.Cu at (161.2, 66.2)
- added D2: 1N4007, Diode_THT:D_DO-41_SOD81_P10.16mm_Horizontal, F.Cu at (144.6, 66.2)
- added D3: 1N4007, Diode_THT:D_DO-41_SOD81_P10.16mm_Horizontal, F.Cu at (142.5, 25.9)
- added J7: Conn_01x06_Pin, Connector_Molex:Molex_KK-254_AE-6410-06A_1x06_P2.54mm_Vertical, F.Cu at (163.9, 84.0)
- added Q1: 2N2222A, 2N2222A:TO92254P470H750-3, F.Cu at (123.4, 51.0)
- added Q2: 2N2222A, 2N2222A:TO92254P470H750-3, F.Cu at (123.4, 58.1)
- added R2: 330, Resistor_THT:R_Axial_DIN0207_L6.3mm_D2.5mm_P10.16mm_Horizontal, F.Cu at (121.3, 50.9)
- added R3: 330, Resistor_THT:R_Axial_DIN0207_L6.3mm_D2.5mm_P10.16mm_Horizontal, F.Cu at (121.0, 57.9)
- added R4: 30k, Resistor_THT:R_Axial_DIN0207_L6.3mm_D2.5mm_P10.16mm_Horizontal, F.Cu at (111.6, 83.1)
- added R5: 330, Resistor_THT:R_Axial_DIN0207_L6.3mm_D2.5mm_P10.16mm_Horizontal, F.Cu at (137.2, 85.5)
- added R6: 330, Resistor_THT:R_Axial_DIN0207_L6.3mm_D2.5mm_P10.16mm_Horizontal, F.Cu at (136.6, 91.5)
- added R7: 30k, Resistor_THT:R_Axial_DIN0207_L6.3mm_D2.5mm_P10.16mm_Horizontal, F.Cu at (111.4, 91.4)
- added U2: PC817, Package_DIP:DIP-4_W7.62mm, F.Cu at (123.0, 85.6)
- added U5: PC817, Package_DIP:DIP-4_W7.62mm, F.Cu at (123.1, 91.4)
- J4: footprint Connector_Molex:Molex_KK-254_AE-6410-03A_1x03_P2.54mm_Vertical -> Connector_Molex:Molex_KK-254_AE-6410-04A_1x04_P2.54mm_Vertical
- J5: footprint Connector_Molex:Molex_KK-254_AE-6410-06A_1x06_P2.54mm_Vertical -> Connector_Molex:Molex_KK-254_AE-6410-07A_1x07_P2.54mm_Vertical
- K1: value rele 3.3v -> SRD-05VDC-SL-C
- K2: value rele 5v -> SRD-05VDC-SL-C
- R1: value 10k -> 30k
- moved U4 140.7 mm to (39.6, 60.7)
- moved J2 139.3 mm to (39.7, 32.6)
- moved C2 67.1 mm to (164.5, 39.5)
- moved C4 67.1 mm to (158.5, 39.5)
- moved C1 67.1 mm to (152.0, 39.5)
- moved C3 67.1 mm to (144.7, 39.5)
- moved U1 67.1 mm to (158.4, 34.0)
- moved U3 67.1 mm to (146.9, 34.0)
- moved J1 66.6 mm to (136.3, 34.8)
- moved R1 58.8 mm to (156.0, 79.7)
- moved K1 58.7 mm to (149.1, 54.5)
- moved J3 58.5 mm to (150.7, 71.3)
- moved J4 58.3 mm to (143.9, 71.3)
- moved K2 57.9 mm to (166.2, 54.5)
- moved J5 55.1 mm to (170.8, 86.6)
Connections:
- C3 pad 1: Net-(J1-Pin_1) -> Net-(D3-K)
- J1 pad 1: Net-(J1-Pin_1) -> Net-(D3-A)
- J3 pad 1: unconnected-(J3-Pin_1-Pad1) -> pin dht
- J4 pad 1: +3.3V sensores -> pin Guva-s12s
- J4 pad 2: GND -> +3.3V sensores
- J4 pad 3: SIG_Guva-s12s -> GND
- J5 pad 5: +5V sensores -> bool ttl
- J5 pad 6: GND -> +5V sensores
- K1 pad A1: vext -> Net-(D2-K)
- K2 pad A1: vext -> Net-(D1-K)
- U3 pad 1: Net-(J1-Pin_1) -> Net-(D3-K)
Routing:
- net GND: track 182.6 -> 263.4 mm
- net +3.3V: track 135.6 -> 65.2 mm
- net bool ttl: track 0.00 -> 52.5 mm
- net RO_TTL: track 63.0 -> 91.9 mm
- net DI_TTL: track 83.9 -> 112.6 mm
- net bool mics: track 0.00 -> 28.7 mm
- net Net-(D1-K): track 0.00 -> 28.5 mm
- net DE/RE_TTL: track 124.5 -> 149.2 mm
- net vext: track 81.4 -> 58.6 mm
- net SIG_Co_MICS-6814: track 72.7 -> 94.5 mm
- net SIG_NH3_MICS-6814: track 66.0 -> 86.7 mm
- net Net-(D3-K): track 0.00 -> 16.3 mm
- net Net-(J1-Pin_1): track 16.1 -> 0.00 mm
- net pin dht: track 0.00 -> 10.7 mm
- net Net-(D2-K): track 0.00 -> 8.02 mm
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- removed copper zone on B.Cu, net GND
Other:
- board outline removed
